Commit message: add reduced pad

File: rh_p12_rn_a_description/urdf/rh_p12_rn_a_gelsight.urdf (robot description, URDF)
Before this commit: robot rh_p12_rn_a, 12 links, 11 joints
Links:
- link rh_p12_rn_base: geometry collision mesh filename=package://rh_p12_rn_gghva_description/meshes/base.stl scale=0.001 0.001 0.001; visual mesh filename=package://rh_p12_rn_a_description/meshes/base.stl scale=0.001 0.001 0.001

Commit message: fiw previous commit and really add reduced pad

File: rh_p12_rn_a_description/urdf/rh_p12_rn_a_gelsight.urdf (robot description, URDF)
Before this commit: robot rh_p12_rn_a, 12 links, 11 joints
Links:
- link rh_p12_rn_base: geometry collision mesh filename=package://rh_p12_rn_a_description/meshes/base.stl scale=0.001 0.001 0.001; visual mesh filename=package://rh_p12_rn_a_description/meshes/base.stl scale=0.001 0.001 0.001
